File: KiCad/TororoKeyboardRightKiCad/TororoKeyboardRightKiCad.sch (KiCad schematic (older format))
At the start: 105 parts, among them J1 MJ-4PP-9, SW1 SW_PUSH, SW10 SW_PUSH, SW11 SW_PUSH, SW12 SW_PUSH, SW13 SW_PUSH, SW14 SW_PUSH, SW15 SW_PUSH, SW16 SW_PUSH, SW17 SW_PUSH, SW18 SW_PUSH, SW19 SW_PUSH, SW2 SW_PUSH, SW20 SW_PUSH, SW21 SW_PUSH, SW22 SW_PUSH, SW23 SW_PUSH, SW24 SW_PUSH, SW25 SW_PUSH, SW26 SW_PUSH, SW27 SW_PUSH, SW28 SW_PUSH, SW29 SW_PUSH, SW3 SW_PUSH, SW30 SW_PUSH, SW31 SW_PUSH, SW32 SW_PUSH, SW33 SW_PUSH, SW34 SW_PUSH, SW4 SW_PUSH, SW5 SW_PUSH, SW6 SW_PUSH, SW7 SW_PUSH, SW8 SW_PUSH, SW9 SW_PUSH, U1 ProMicro

Commit message: 右手側のレイアウト作成
TODO: 配線
Parts:
- D10, D15, D2, D3, D4, D5: footprint (none) -> kbd_tororo:D3_TH_SMD_top
- SW10, SW15, SW2, SW3, SW4, SW5: footprint (none) -> kbd_tororo:Hybrid_PCB_100H_no-silk_no_ref
Changed lines of the file:
@@
 EESchema Schematic File Version 4
+LIBS:TororoKeyboardRightKiCad-cache
 EELAYER 29 0
 EELAYER END
@@
 F 0 "SW2" H 3200 3505 50  0000 C CNN
 F 1 "SW_PUSH" H 3200 3414 50  0000 C CNN
-F 2 "" H 3200 3250 50  0000 C CNN
+F 2 "kbd_tororo:Hybrid_PCB_100H_no-silk_no_ref" H 3200 3250 50  0001 C CNN
 F 3 "" H 3200 3250 50  0000 C CNN
 	1    3200 3250
@@
 F 0 "SW3" H 3200 4255 50  0000 C CNN
 F 1 "SW_PUSH" H 3200 4164 50  0000 C CNN
-F 2 "" H 3200 4000 50  0000 C CNN
+F 2 "kbd_tororo:Hybrid_PCB_100H_no-silk_no_ref" H 3200 4000 50  0001 C CNN
 F 3 "" H 3200 4000 50  0000 C CNN
 	1    3200 4000
@@
 F 0 "SW4" H 3200 5005 50  0000 C CNN
 F 1 "SW_PUSH" H 3200 4914 50  0000 C CNN
-F 2 "" H 3200 4750 50  0000 C CNN
+F 2 "kbd_tororo:Hybrid_PCB_100H_no-silk_no_ref" H 3200 4750 50  0001 C CNN
 F 3 "" H 3200 4750 50  0000 C CNN
 	1    3200 4750
@@
 F 0 "SW5" H 3200 5755 50  0000 C CNN
 F 1 "SW_PUSH" H 3200 5664 50  0000 C CNN
-F 2 "" H 3200 5500 50  0000 C CNN
+F 2 "kbd_tororo:Hybrid_PCB_100H_no-silk_no_ref" H 3200 5500 50  0001 C CNN
 F 3 "" H 3200 5500 50  0000 C CNN
 	1    3200 5500
@@
 F 0 "SW10" H 4200 5755 50  0000 C CNN
 F 1 "SW_PUSH" H 4200 5664 50  0000 C CNN
-F 2 "" H 4200 5500 50  0000 C CNN
+F 2 "kbd_tororo:Hybrid_PCB_100H_no-silk_no_ref" H 4200 5500 50  0001 C CNN
 F 3 "" H 4200 5500 50  0000 C CNN
 	1    4200 5500
@@
 F 0 "SW15" H 5200 5755 50  0000 C CNN
 F 1 "SW_PUSH" H 5200 5664 50  0000 C CNN
-F 2 "" H 5200 5500 50  0000 C CNN
+F 2 "kbd_tororo:Hybrid_PCB_100H_no-silk_no_ref" H 5200 5500 50  0001 C CNN
 F 3 "" H 5200 5500 50  0000 C CNN
 	1    5200 5500
@@
 F 0 "D2" V 3546 3321 50  0000 R CNN
 F 1 "D" V 3455 3321 50  0000 R CNN
-F 2 "" H 3500 3400 50  0001 C CNN
+F 2 "kbd_tororo:D3_TH_SMD_top" H 3500 3400 50  0001 C CNN
 F 3 "~" H 3500 3400 50  0001 C CNN
 	1    3500 3400
@@
 F 0 "D3" V 3546 4071 50  0000 R CNN
 F 1 "D" V 3455 4071 50  0000 R CNN
-F 2 "" H 3500 4150 50  0001 C CNN
+F 2 "kbd_tororo:D3_TH_SMD_top" H 3500 4150 50  0001 C CNN
 F 3 "~" H 3500 4150 50  0001 C CNN
 	1    3500 4150
@@
 F 0 "D4" V 3546 4821 50  0000 R CNN
 F 1 "D" V 3455 4821 50  0000 R CNN
-F 2 "" H 3500 4900 50  0001 C CNN
+F 2 "kbd_tororo:D3_TH_SMD_top" H 3500 4900 50  0001 C CNN
 F 3 "~" H 3500 4900 50  0001 C CNN
 	1    3500 4900
@@
 F 0 "D5" V 3546 5571 50  0000 R CNN
 F 1 "D" V 3455 5571 50  0000 R CNN
-F 2 "" H 3500 5650 50  0001 C CNN
+F 2 "kbd_tororo:D3_TH_SMD_top" H 3500 5650 50  0001 C CNN
 F 3 "~" H 3500 5650 50  0001 C CNN
 	1    3500 5650
@@
 F 0 "D10" V 4546 5571 50  0000 R CNN
 F 1 "D" V 4455 5571 50  0000 R CNN
-F 2 "" H 4500 5650 50  0001 C CNN
+F 2 "kbd_tororo:D3_TH_SMD_top" H 4500 5650 50  0001 C CNN
 F 3 "~" H 4500 5650 50  0001 C CNN
 	1    4500 5650
@@
 F 0 "D15" V 5546 5571 50  0000 R CNN
 F 1 "D" V 5455 5571 50  0000 R CNN
-F 2 "" H 5500 5650 50  0001 C CNN
+F 2 "kbd_tororo:D3_TH_SMD_top" H 5500 5650 50  0001 C CNN
 F 3 "~" H 5500 5650 50  0001 C CNN
 	1    5500 5650

Commit message: pro micro のフットプリントを右手用に修正してレイアウトを更新
文字の位置を変更した。
Parts:
- U1: footprint kbd_tororo:ProMicro_v2_back -> kbd_tororo:ProMicro_v2_back_right
Changed lines of the file:
@@
 F 0 "U1" H 13000 5387 60  0000 C CNN
 F 1 "ProMicro" H 13000 5281 60  0000 C CNN
-F 2 "kbd_tororo:ProMicro_v2_back" H 13100 3300 60  0001 C CNN
+F 2 "kbd_tororo:ProMicro_v2_back_right" H 13100 3300 60  0001 C CNN
 F 3 "" H 13100 3300 60  0000 C CNN
 	1    13000 4350
