File: KiCad/TororoKeyboardLeftKiCad/TororoKeyboardLeftKiCad.kicad_pcb (KiCad board)
At the start: 2 copper layers, 139.7 x 99.2 mm, 97 parts, among them J1 MJ-4PP-9, SW1 SW_PUSH, SW10 SW_PUSH, SW11 SW_PUSH, SW12 SW_PUSH, SW13 SW_PUSH, SW14 SW_PUSH, SW15 SW_PUSH, SW16 SW_PUSH, SW17 SW_PUSH, SW18 SW_PUSH, SW19 SW_PUSH, SW2 SW_PUSH, SW20 SW_PUSH, SW21 SW_PUSH, SW22 SW_PUSH, SW23 SW_PUSH, SW24 SW_PUSH, SW25 SW_PUSH, SW26 SW_PUSH, SW27 SW_PUSH, SW28 SW_PUSH, SW29 SW_PUSH, SW3 SW_PUSH, SW4 SW_PUSH, SW5 SW_PUSH, SW6 SW_PUSH, SW7 SW_PUSH, SW8 SW_PUSH, SW9 SW_PUSH, U1 ProMicro

Commit message: 左手側の配線を再度修正
Routing:
- net VCC: track 875.2 -> 885.6 mm, vias 11 -> 47
- net col3: track 108.1 -> 110.0 mm
- net col6: track 184.2 -> 185.8 mm
- net col5: track 176.9 -> 178.4 mm
- net col4: track 183.9 -> 185.4 mm
- net Net-(D26-Pad2): track 14.2 -> 15.1 mm, vias 0 -> 1
- net Net-(L24-Pad3): track 26.9 -> 27.4 mm
- net GND: vias 24 -> 31
- net (no net): vias 0 -> 1
